File: pcb/keyboard_pcb.kicad_sch (KiCad schematic)
At the start: 23 parts, among them J1 TRRS, K00 KEYSW, K01 KEYSW, K02 KEYSW, K03 KEYSW, K04 KEYSW, K05 KEYSW, K10 KEYSW, K11 KEYSW, K12 KEYSW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

Commit message: Added speaker
Parts:
- added LS1: AST1109MLTRQ, ergodonk_kicad_library:AST1109MLTRQ, symbol AST1109MLTRQ:AST1109MLTRQ
- J1: footprint Keebio-Parts:TRRS-PJ-320A -> ergodonk_kicad_library:MJ-4PP-9_CANTOR_KITCHEN_SINK
- K00, K01, K02, K03, K04, K05, K10, K11, K12, K13, K14, K15, K20, K21, K22, K23, K24, K25, K30, K31, K32: footprint keyswitches:SW_PG1350_reversible -> ergodonk_kicad_library:ALL LOWs CANTOR
- U1: footprint Footprints:YAAJ_WeAct_BlackPill_2 -> ergodonk_kicad_library:Cantor_DS_YAAJ_WeAct_BlackPill_2
Connections:
- net GND: now also LS1.2
- net AUDIO: now reaches U1.1 (PB12)
- net AUDIO: now also LS1.1
- no-connect marks 13 -> 12
Other:
- note added: "Speaker"
- note added: "https://docs.qmk.fm/#/feature_audio?id=pwm-software"

Commit message: Updated switch footrpints
Parts:
- J1: footprint ergodonk_kicad_library:MJ-4PP-9_CANTOR_KITCHEN_SINK -> Cantor_MasterKey:MJ-4PP-9_CANTOR_KITCHEN_SINK
- K00, K01, K02, K03, K04, K05, K10, K11, K12, K13, K14, K15, K20, K21, K22, K23, K24, K25, K30, K31, K32: footprint ergodonk_kicad_library:ALL LOWs CANTOR -> Cantor_MasterKey:ALL LOWs CANTOR
- LS1: value AST1109MLTRQ -> AST1109MLTRQ_MAL; footprint ergodonk_kicad_library:AST1109MLTRQ -> Cantor_MasterKey:AST1109MLTRQ
- U1: footprint ergodonk_kicad_library:Cantor_DS_YAAJ_WeAct_BlackPill_2 -> Cantor_MasterKey:Cantor_DS_YAAJ_WeAct_BlackPill_2
Changed lines of the file:
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@@
       (effects (font (size 1.524 1.524)) hide)
     )
-    (property "Footprint" "ergodonk_kicad_library:ALL LOWs CANTOR" (at 264.16 76.2 0)
+    (property "Footprint" "Cantor_MasterKey:ALL LOWs CANTOR" (at 264.16 76.2 0)
       (effects (font (size 1.524 1.524)) hide)
     )
@@
       (effects (font (size 1.524 1.524)) hide)
     )
-    (property "Footprint" "ergodonk_kicad_library:ALL LOWs CANTOR" (at 238.76 60.96 0)
+    (property "Footprint" "Cantor_MasterKey:ALL LOWs CANTOR" (at 238.76 60.96 0)
       (effects (font (size 1.524 1.524)) hide)
     )
@@
       (effects (font (size 1.524 1.524)) hide)
     )
-    (property "Footprint" "ergodonk_kicad_library:ALL LOWs CANTOR" (at 137.16 30.48 0)
+    (property "Footprint" "Cantor_MasterKey:ALL LOWs CANTOR" (at 137.16 30.48 0)
       (effects (font (size 1.524 1.524)) hide)
     )
@@
       (effects (font (size 1.524 1.524)) hide)
     )
-    (property "Footprint" "ergodonk_kicad_library:ALL LOWs CANTOR" (at 264.16 45.72 0)
+    (property "Footprint" "Cantor_MasterKey:ALL LOWs CANTOR" (at 264.16 45.72 0)
       (effects (font (size 1.524 1.524)) hide)
     )
@@
       (effects (font (size 1.524 1.524)) hide)
     )
-    (property "Footprint" "ergodonk_kicad_library:ALL LOWs CANTOR" (at 213.36 30.48 0)
+    (property "Footprint" "Cantor_MasterKey:ALL LOWs CANTOR" (at 213.36 30.48 0)
       (effects (font (size 1.524 1.524)) hide)
     )
@@
       (effects (font (size 1.524 1.524)) hide)
     )
-    (property "Footprint" "ergodonk_kicad_library:ALL LOWs CANTOR" (at 187.96 30.48 0)
+    (property "Footprint" "Cantor_MasterKey:ALL LOWs CANTOR" (at 187.96 30.48 0)
       (effects (font (size 1.524 1.524)) hide)
     )
@@
       (effects (font (size 1.524 1.524)) hide)
     )
-    (property "Footprint" "ergodonk_kicad_library:ALL LOWs CANTOR" (at 162.56 45.72 0)
+    (property "Footprint" "Cantor_MasterKey:ALL LOWs CANTOR" (at 162.56 45.72 0)
       (effects (font (size 1.524 1.524)) hide)
     )
@@
       (effects (font (size 1.524 1.524)) hide)
     )
-    (property "Footprint" "ergodonk_kicad_library:ALL LOWs CANTOR" (at 187.96 60.96 0)
+    (property "Footprint" "Cantor_MasterKey:ALL LOWs CANTOR" (at 187.96 60.96 0)
       (effects (font (size 1.524 1.524)) hide)
     )
@@
       (effects (font (size 1.27 1.27)))
     )
-    (property "Footprint" "ergodonk_kicad_library:Cantor_DS_YAAJ_WeAct_BlackPill_2" (at 71.374 87.122 0)
+    (property "Footprint" "Cantor_MasterKey:Cantor_DS_YAAJ_WeAct_BlackPill_2" (at 71.374 87.122 0)
       (effects (font (size 1.27 1.27)) hide)
     )
@@
       (effects (font (size 1.524 1.524)) (justify left))
     )
-    (property "Value" "AST1109MLTRQ" (at 110.49 121.92 0)
+    (property "Value" "AST1109MLTRQ_MAL" (at 110.49 121.92 0)
       (effects (font (size 1.524 1.524)) (justify left))
     )
-    (property "Footprint" "ergodonk_kicad_library:AST1109MLTRQ" (at 101.6 114.554 0)
+    (property "Footprint" "Cantor_MasterKey:AST1109MLTRQ" (at 101.6 114.554 0)
       (effects (font (size 1.524 1.524)) hide)
     )
@@
       (effects (font (size 1.524 1.524)) hide)
     )
-    (property "Footprint" "ergodonk_kicad_library:ALL LOWs CANTOR" (at 238.76 30.48 0)
+    (property "Footprint" "Cantor_MasterKey:ALL LOWs CANTOR" (at 238.76 30.48 0)
       (effects (font (size 1.524 1.524)) hide)
     )
@@
       (effects (font (size 1.524 1.524)) hide)
     )
-    (property "Footprint" "ergodonk_kicad_library:ALL LOWs CANTOR" (at 213.36 76.2 0)
+    (property "Footprint" "Cantor_MasterKey:ALL LOWs CANTOR" (at 213.36 76.2 0)
       (effects (font (size 1.524 1.524)) hide)
     )
@@
       (effects (font (size 1.524 1.524)))
     )
-    (property "Footprint" "ergodonk_kicad_library:MJ-4PP-9_CANTOR_KITCHEN_SINK" (at 46.99 115.57 0)
+    (property "Footprint" "Cantor_MasterKey:MJ-4PP-9_CANTOR_KITCHEN_SINK" (at 46.99 115.57 0)
       (effects (font (size 1.524 1.524)) hide)
     )
@@
       (effects (font (size 1.524 1.524)) hide)
     )
-    (property "Footprint" "ergodonk_kicad_library:ALL LOWs CANTOR" (at 137.16 60.96 0)
+    (property "Footprint" "Cantor_MasterKey:ALL LOWs CANTOR" (at 137.16 60.96 0)
       (effects (font (size 1.524 1.524)) hide)
     )
@@
       (effects (font (size 1.524 1.524)) hide)
     )
-    (property "Footprint" "ergodonk_kicad_library:ALL LOWs CANTOR" (at 213.36 60.96 0)
+    (property "Footprint" "Cantor_MasterKey:ALL LOWs CANTOR" (at 213.36 60.96 0)
       (effects (font (size 1.524 1.524)) hide)
     )
@@
       (effects (font (size 1.524 1.524)) hide)
     )
-    (property "Footprint" "ergodonk_kicad_library:ALL LOWs CANTOR" (at 137.16 45.72 0)
+    (property "Footprint" "Cantor_MasterKey:ALL LOWs CANTOR" (at 137.16 45.72 0)
       (effects (font (size 1.524 1.524)) hide)
     )
@@
       (effects (font (size 1.524 1.524)) hide)
     )
-    (property "Footprint" "ergodonk_kicad_library:ALL LOWs CANTOR" (at 162.56 30.48 0)
+    (property "Footprint" "Cantor_MasterKey:ALL LOWs CANTOR" (at 162.56 30.48 0)
       (effects (font (size 1.524 1.524)) hide)
     )
@@
       (effects (font (size 1.524 1.524)) hide)
     )
-    (property "Footprint" "ergodonk_kicad_library:ALL LOWs CANTOR" (at 264.16 60.96 0)
+    (property "Footprint" "Cantor_MasterKey:ALL LOWs CANTOR" (at 264.16 60.96 0)
       (effects (font (size 1.524 1.524)) hide)
     )
@@
       (effects (font (size 1.524 1.524)) hide)
     )
-    (property "Footprint" "ergodonk_kicad_library:ALL LOWs CANTOR" (at 238.76 76.2 0)
+    (property "Footprint" "Cantor_MasterKey:ALL LOWs CANTOR" (at 238.76 76.2 0)
       (effects (font (size 1.524 1.524)) hide)
     )
@@
       (effects (font (size 1.524 1.524)) hide)
     )
-    (property "Footprint" "ergodonk_kicad_library:ALL LOWs CANTOR" (at 238.76 45.72 0)
+    (property "Footprint" "Cantor_MasterKey:ALL LOWs CANTOR" (at 238.76 45.72 0)
       (effects (font (size 1.524 1.524)) hide)
     )
@@
       (effects (font (size 1.524 1.524)) hide)
     )
-    (property "Footprint" "ergodonk_kicad_library:ALL LOWs CANTOR" (at 213.36 45.72 0)
+    (property "Footprint" "Cantor_MasterKey:ALL LOWs CANTOR" (at 213.36 45.72 0)
       (effects (font (size 1.524 1.524)) hide)
     )
@@
       (effects (font (size 1.524 1.524)) hide)
     )
-    (property "Footprint" "ergodonk_kicad_library:ALL LOWs CANTOR" (at 162.56 60.96 0)
+    (property "Footprint" "Cantor_MasterKey:ALL LOWs CANTOR" (at 162.56 60.96 0)
       (effects (font (size 1.524 1.524)) hide)
     )
@@
       (effects (font (size 1.524 1.524)) hide)
     )
-    (property "Footprint" "ergodonk_kicad_library:ALL LOWs CANTOR" (at 187.96 45.72 0)
+    (property "Footprint" "Cantor_MasterKey:ALL LOWs CANTOR" (at 187.96 45.72 0)
       (effects (font (size 1.524 1.524)) hide)
     )
@@
       (effects (font (size 1.524 1.524)) hide)
     )
-    (property "Footprint" "ergodonk_kicad_library:ALL LOWs CANTOR" (at 264.16 30.48 0)
-      (effects (font (size 1.524 1.524)) hide)
-    )
+    (property "Footprint" "Cantor_MasterKey:ALL LOWs CANTOR" (at 264.16 30.48 0)
+      (effects (font (size 1.524 1.524)) hide)
+    )

Commit message: Fixed choc 2nd min misalingment Revised 'everything' footprint: combined red-dragon and MX hole removed organic masks in leiu of exotic annular rings fixed malformed edge shapes
Parts:
- K00, K01, K02, K03, K04, K05, K10, K11, K12, K13, K14, K15, K20, K21, K22, K23, K24, K25, K30, K31, K32: footprint Cantor_MasterKey:ALL LOWs CANTOR -> Cantor_MasterKey:ALL LOWs CANTOR v4.1
Changed lines of the file:
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@@
       (effects (font (size 1.524 1.524)) hide)
     )
-    (property "Footprint" "Cantor_MasterKey:ALL LOWs CANTOR" (at 264.16 76.2 0)
+    (property "Footprint" "Cantor_MasterKey:ALL LOWs CANTOR v4.1" (at 264.16 76.2 0)
       (effects (font (size 1.524 1.524)) hide)
     )
@@
       (effects (font (size 1.524 1.524)) hide)
     )
-    (property "Footprint" "Cantor_MasterKey:ALL LOWs CANTOR" (at 238.76 60.96 0)
+    (property "Footprint" "Cantor_MasterKey:ALL LOWs CANTOR v4.1" (at 238.76 60.96 0)
       (effects (font (size 1.524 1.524)) hide)
     )
@@
       (effects (font (size 1.524 1.524)) hide)
     )
-    (property "Footprint" "Cantor_MasterKey:ALL LOWs CANTOR" (at 137.16 30.48 0)
+    (property "Footprint" "Cantor_MasterKey:ALL LOWs CANTOR v4.1" (at 137.16 30.48 0)
       (effects (font (size 1.524 1.524)) hide)
     )
@@
       (effects (font (size 1.524 1.524)) hide)
     )
-    (property "Footprint" "Cantor_MasterKey:ALL LOWs CANTOR" (at 264.16 45.72 0)
+    (property "Footprint" "Cantor_MasterKey:ALL LOWs CANTOR v4.1" (at 264.16 45.72 0)
       (effects (font (size 1.524 1.524)) hide)
     )
@@
       (effects (font (size 1.524 1.524)) hide)
     )
-    (property "Footprint" "Cantor_MasterKey:ALL LOWs CANTOR" (at 213.36 30.48 0)
+    (property "Footprint" "Cantor_MasterKey:ALL LOWs CANTOR v4.1" (at 213.36 30.48 0)
       (effects (font (size 1.524 1.524)) hide)
     )
@@
       (effects (font (size 1.524 1.524)) hide)
     )
-    (property "Footprint" "Cantor_MasterKey:ALL LOWs CANTOR" (at 187.96 30.48 0)
+    (property "Footprint" "Cantor_MasterKey:ALL LOWs CANTOR v4.1" (at 187.96 30.48 0)
       (effects (font (size 1.524 1.524)) hide)
     )
@@
       (effects (font (size 1.524 1.524)) hide)
     )
-    (property "Footprint" "Cantor_MasterKey:ALL LOWs CANTOR" (at 162.56 45.72 0)
+    (property "Footprint" "Cantor_MasterKey:ALL LOWs CANTOR v4.1" (at 162.56 45.72 0)
       (effects (font (size 1.524 1.524)) hide)
     )
@@
       (effects (font (size 1.524 1.524)) hide)
     )
-    (property "Footprint" "Cantor_MasterKey:ALL LOWs CANTOR" (at 187.96 60.96 0)
+    (property "Footprint" "Cantor_MasterKey:ALL LOWs CANTOR v4.1" (at 187.96 60.96 0)
       (effects (font (size 1.524 1.524)) hide)
     )
@@
       (effects (font (size 1.524 1.524)) hide)
     )
-    (property "Footprint" "Cantor_MasterKey:ALL LOWs CANTOR" (at 238.76 30.48 0)
+    (property "Footprint" "Cantor_MasterKey:ALL LOWs CANTOR v4.1" (at 238.76 30.48 0)
       (effects (font (size 1.524 1.524)) hide)
     )
@@
       (effects (font (size 1.524 1.524)) hide)
     )
-    (property "Footprint" "Cantor_MasterKey:ALL LOWs CANTOR" (at 213.36 76.2 0)
+    (property "Footprint" "Cantor_MasterKey:ALL LOWs CANTOR v4.1" (at 213.36 76.2 0)
       (effects (font (size 1.524 1.524)) hide)
     )
@@
       (effects (font (size 1.524 1.524)) hide)
     )
-    (property "Footprint" "Cantor_MasterKey:ALL LOWs CANTOR" (at 137.16 60.96 0)
+    (property "Footprint" "Cantor_MasterKey:ALL LOWs CANTOR v4.1" (at 137.16 60.96 0)
       (effects (font (size 1.524 1.524)) hide)
     )
@@
       (effects (font (size 1.524 1.524)) hide)
     )
-    (property "Footprint" "Cantor_MasterKey:ALL LOWs CANTOR" (at 213.36 60.96 0)
+    (property "Footprint" "Cantor_MasterKey:ALL LOWs CANTOR v4.1" (at 213.36 60.96 0)
       (effects (font (size 1.524 1.524)) hide)
     )
@@
       (effects (font (size 1.524 1.524)) hide)
     )
-    (property "Footprint" "Cantor_MasterKey:ALL LOWs CANTOR" (at 137.16 45.72 0)
+    (property "Footprint" "Cantor_MasterKey:ALL LOWs CANTOR v4.1" (at 137.16 45.72 0)
       (effects (font (size 1.524 1.524)) hide)
     )
@@
       (effects (font (size 1.524 1.524)) hide)
     )
-    (property "Footprint" "Cantor_MasterKey:ALL LOWs CANTOR" (at 162.56 30.48 0)
+    (property "Footprint" "Cantor_MasterKey:ALL LOWs CANTOR v4.1" (at 162.56 30.48 0)
       (effects (font (size 1.524 1.524)) hide)
     )
@@
       (effects (font (size 1.524 1.524)) hide)
     )
-    (property "Footprint" "Cantor_MasterKey:ALL LOWs CANTOR" (at 264.16 60.96 0)
+    (property "Footprint" "Cantor_MasterKey:ALL LOWs CANTOR v4.1" (at 264.16 60.96 0)
       (effects (font (size 1.524 1.524)) hide)
     )
@@
       (effects (font (size 1.524 1.524)) hide)
     )
-    (property "Footprint" "Cantor_MasterKey:ALL LOWs CANTOR" (at 238.76 76.2 0)
+    (property "Footprint" "Cantor_MasterKey:ALL LOWs CANTOR v4.1" (at 238.76 76.2 0)
       (effects (font (size 1.524 1.524)) hide)
     )
@@
       (effects (font (size 1.524 1.524)) hide)
     )
-    (property "Footprint" "Cantor_MasterKey:ALL LOWs CANTOR" (at 238.76 45.72 0)
+    (property "Footprint" "Cantor_MasterKey:ALL LOWs CANTOR v4.1" (at 238.76 45.72 0)
       (effects (font (size 1.524 1.524)) hide)
     )
@@
       (effects (font (size 1.524 1.524)) hide)
     )
-    (property "Footprint" "Cantor_MasterKey:ALL LOWs CANTOR" (at 213.36 45.72 0)
+    (property "Footprint" "Cantor_MasterKey:ALL LOWs CANTOR v4.1" (at 213.36 45.72 0)
       (effects (font (size 1.524 1.524)) hide)
     )
@@
       (effects (font (size 1.524 1.524)) hide)
     )
-    (property "Footprint" "Cantor_MasterKey:ALL LOWs CANTOR" (at 162.56 60.96 0)
+    (property "Footprint" "Cantor_MasterKey:ALL LOWs CANTOR v4.1" (at 162.56 60.96 0)
       (effects (font (size 1.524 1.524)) hide)
     )
@@
       (effects (font (size 1.524 1.524)) hide)
     )
-    (property "Footprint" "Cantor_MasterKey:ALL LOWs CANTOR" (at 187.96 45.72 0)
+    (property "Footprint" "Cantor_MasterKey:ALL LOWs CANTOR v4.1" (at 187.96 45.72 0)
       (effects (font (size 1.524 1.524)) hide)
     )
@@
       (effects (font (size 1.524 1.524)) hide)
     )
-    (property "Footprint" "Cantor_MasterKey:ALL LOWs CANTOR" (at 264.16 30.48 0)
-      (effects (font (size 1.524 1.524)) hide)
-    )
+    (property "Footprint" "Cantor_MasterKey:ALL LOWs CANTOR v4.1" (at 264.16 30.48 0)
+      (effects (font (size 1.524 1.524)) hide)
+    )

Commit message: Updated docs and fixed footprint mask
Parts:
- K00, K01, K02, K03, K04, K05, K10, K11, K12, K13, K14, K15, K20, K21, K22, K23, K24, K25, K30, K31, K32: footprint Cantor_MasterKey:ALL LOWs CANTOR v4.1 -> Cantor_MasterKey:CherryMX_ChocV2_1u_DS
Changed lines of the file:
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@@
       (effects (font (size 1.524 1.524)) hide)
     )
-    (property "Footprint" "Cantor_MasterKey:ALL LOWs CANTOR v4.1" (at 264.16 76.2 0)
+    (property "Footprint" "Cantor_MasterKey:CherryMX_ChocV2_1u_DS" (at 264.16 76.2 0)
       (effects (font (size 1.524 1.524)) hide)
     )
@@
       (effects (font (size 1.524 1.524)) hide)
     )
-    (property "Footprint" "Cantor_MasterKey:ALL LOWs CANTOR v4.1" (at 238.76 60.96 0)
+    (property "Footprint" "Cantor_MasterKey:CherryMX_ChocV2_1u_DS" (at 238.76 60.96 0)
       (effects (font (size 1.524 1.524)) hide)
     )
@@
       (effects (font (size 1.524 1.524)) hide)
     )
-    (property "Footprint" "Cantor_MasterKey:ALL LOWs CANTOR v4.1" (at 137.16 30.48 0)
+    (property "Footprint" "Cantor_MasterKey:CherryMX_ChocV2_1u_DS" (at 137.16 30.48 0)
       (effects (font (size 1.524 1.524)) hide)
     )
@@
       (effects (font (size 1.524 1.524)) hide)
     )
-    (property "Footprint" "Cantor_MasterKey:ALL LOWs CANTOR v4.1" (at 264.16 45.72 0)
+    (property "Footprint" "Cantor_MasterKey:CherryMX_ChocV2_1u_DS" (at 264.16 45.72 0)
       (effects (font (size 1.524 1.524)) hide)
     )
@@
       (effects (font (size 1.524 1.524)) hide)
     )
-    (property "Footprint" "Cantor_MasterKey:ALL LOWs CANTOR v4.1" (at 213.36 30.48 0)
+    (property "Footprint" "Cantor_MasterKey:CherryMX_ChocV2_1u_DS" (at 213.36 30.48 0)
       (effects (font (size 1.524 1.524)) hide)
     )
@@
       (effects (font (size 1.524 1.524)) hide)
     )
-    (property "Footprint" "Cantor_MasterKey:ALL LOWs CANTOR v4.1" (at 187.96 30.48 0)
+    (property "Footprint" "Cantor_MasterKey:CherryMX_ChocV2_1u_DS" (at 187.96 30.48 0)
       (effects (font (size 1.524 1.524)) hide)
     )
@@
       (effects (font (size 1.524 1.524)) hide)
     )
-    (property "Footprint" "Cantor_MasterKey:ALL LOWs CANTOR v4.1" (at 162.56 45.72 0)
+    (property "Footprint" "Cantor_MasterKey:CherryMX_ChocV2_1u_DS" (at 162.56 45.72 0)
       (effects (font (size 1.524 1.524)) hide)
     )
@@
       (effects (font (size 1.524 1.524)) hide)
     )
-    (property "Footprint" "Cantor_MasterKey:ALL LOWs CANTOR v4.1" (at 187.96 60.96 0)
+    (property "Footprint" "Cantor_MasterKey:CherryMX_ChocV2_1u_DS" (at 187.96 60.96 0)
       (effects (font (size 1.524 1.524)) hide)
     )
@@
       (effects (font (size 1.524 1.524)) hide)
     )
-    (property "Footprint" "Cantor_MasterKey:ALL LOWs CANTOR v4.1" (at 238.76 30.48 0)
+    (property "Footprint" "Cantor_MasterKey:CherryMX_ChocV2_1u_DS" (at 238.76 30.48 0)
       (effects (font (size 1.524 1.524)) hide)
     )
@@
       (effects (font (size 1.524 1.524)) hide)
     )
-    (property "Footprint" "Cantor_MasterKey:ALL LOWs CANTOR v4.1" (at 213.36 76.2 0)
+    (property "Footprint" "Cantor_MasterKey:CherryMX_ChocV2_1u_DS" (at 213.36 76.2 0)
       (effects (font (size 1.524 1.524)) hide)
     )
@@
       (effects (font (size 1.524 1.524)) hide)
     )
-    (property "Footprint" "Cantor_MasterKey:ALL LOWs CANTOR v4.1" (at 137.16 60.96 0)
+    (property "Footprint" "Cantor_MasterKey:CherryMX_ChocV2_1u_DS" (at 137.16 60.96 0)
       (effects (font (size 1.524 1.524)) hide)
     )
@@
       (effects (font (size 1.524 1.524)) hide)
     )
-    (property "Footprint" "Cantor_MasterKey:ALL LOWs CANTOR v4.1" (at 213.36 60.96 0)
+    (property "Footprint" "Cantor_MasterKey:CherryMX_ChocV2_1u_DS" (at 213.36 60.96 0)
       (effects (font (size 1.524 1.524)) hide)
     )
@@
       (effects (font (size 1.524 1.524)) hide)
     )
-    (property "Footprint" "Cantor_MasterKey:ALL LOWs CANTOR v4.1" (at 137.16 45.72 0)
+    (property "Footprint" "Cantor_MasterKey:CherryMX_ChocV2_1u_DS" (at 137.16 45.72 0)
       (effects (font (size 1.524 1.524)) hide)
     )
@@
       (effects (font (size 1.524 1.524)) hide)
     )
-    (property "Footprint" "Cantor_MasterKey:ALL LOWs CANTOR v4.1" (at 162.56 30.48 0)
+    (property "Footprint" "Cantor_MasterKey:CherryMX_ChocV2_1u_DS" (at 162.56 30.48 0)
       (effects (font (size 1.524 1.524)) hide)
     )
@@
       (effects (font (size 1.524 1.524)) hide)
     )
-    (property "Footprint" "Cantor_MasterKey:ALL LOWs CANTOR v4.1" (at 264.16 60.96 0)
+    (property "Footprint" "Cantor_MasterKey:CherryMX_ChocV2_1u_DS" (at 264.16 60.96 0)
       (effects (font (size 1.524 1.524)) hide)
     )
@@
       (effects (font (size 1.524 1.524)) hide)
     )
-    (property "Footprint" "Cantor_MasterKey:ALL LOWs CANTOR v4.1" (at 238.76 76.2 0)
+    (property "Footprint" "Cantor_MasterKey:CherryMX_ChocV2_1u_DS" (at 238.76 76.2 0)
       (effects (font (size 1.524 1.524)) hide)
     )
@@
       (effects (font (size 1.524 1.524)) hide)
     )
-    (property "Footprint" "Cantor_MasterKey:ALL LOWs CANTOR v4.1" (at 238.76 45.72 0)
+    (property "Footprint" "Cantor_MasterKey:CherryMX_ChocV2_1u_DS" (at 238.76 45.72 0)
       (effects (font (size 1.524 1.524)) hide)
     )
@@
       (effects (font (size 1.524 1.524)) hide)
     )
-    (property "Footprint" "Cantor_MasterKey:ALL LOWs CANTOR v4.1" (at 213.36 45.72 0)
+    (property "Footprint" "Cantor_MasterKey:CherryMX_ChocV2_1u_DS" (at 213.36 45.72 0)
       (effects (font (size 1.524 1.524)) hide)
     )
@@
       (effects (font (size 1.524 1.524)) hide)
     )
-    (property "Footprint" "Cantor_MasterKey:ALL LOWs CANTOR v4.1" (at 162.56 60.96 0)
+    (property "Footprint" "Cantor_MasterKey:CherryMX_ChocV2_1u_DS" (at 162.56 60.96 0)
       (effects (font (size 1.524 1.524)) hide)
     )
@@
       (effects (font (size 1.524 1.524)) hide)
     )
-    (property "Footprint" "Cantor_MasterKey:ALL LOWs CANTOR v4.1" (at 187.96 45.72 0)
+    (property "Footprint" "Cantor_MasterKey:CherryMX_ChocV2_1u_DS" (at 187.96 45.72 0)
       (effects (font (size 1.524 1.524)) hide)
     )
@@
       (effects (font (size 1.524 1.524)) hide)
     )
-    (property "Footprint" "Cantor_MasterKey:ALL LOWs CANTOR v4.1" (at 264.16 30.48 0)
-      (effects (font (size 1.524 1.524)) hide)
-    )
+    (property "Footprint" "Cantor_MasterKey:CherryMX_ChocV2_1u_DS" (at 264.16 30.48 0)
+      (effects (font (size 1.524 1.524)) hide)
+    )

Commit message: Fixed trrs footprint added key numbering cleaned up wiring between blackpill holes
Parts:
- J1: footprint Cantor_MasterKey:MJ-4PP-9_CANTOR_KITCHEN_SINK -> Cantor_MasterKey:MJ-4PP-9_Cantor_MX_TX-RX_Crossover
Changed lines of the file:
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@@
       (effects (font (size 1.524 1.524)))
     )
-    (property "Footprint" "Cantor_MasterKey:MJ-4PP-9_CANTOR_KITCHEN_SINK" (at 46.99 115.57 0)
+    (property "Footprint" "Cantor_MasterKey:MJ-4PP-9_Cantor_MX_TX-RX_Crossover" (at 46.99 115.57 0)
       (effects (font (size 1.524 1.524)) hide)
     )
