File: pcb/keyboard_pcb.kicad_sch (KiCad schematic)
At the start: 24 parts, among them J1 TRRS, K00 KEYSW, K01 KEYSW, K02 KEYSW, K03 KEYSW, K04 KEYSW, K05 KEYSW, K10 KEYSW, K11 KEYSW, K12 KEYSW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

Commit message: Removed speaker
Parts:
- removed LS1: AST1109MLTRQ_MAL, Cantor_MasterKey:AST1109MLTRQ, symbol AST1109MLTRQ:AST1109MLTRQ
Connections:
- net AUDIO: no longer names the net of U1.1 (PB12)
- no-connect marks 12 -> 13
Other:
- note removed: "Speaker"
Changed lines of the file:
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@@
   (no_connect (at 91.44 34.29))
   (no_connect (at 50.8 77.47))
+  (no_connect (at 50.8 34.29))
   (wire (pts (xy 149.86 60.96) (xy 154.94 60.96))
     (stroke (width 0) (type default))
@@
     (stroke (width 0) (type default))
   )
-  (wire (pts (xy 93.98 121.92) (xy 93.98 120.65))
-    (stroke (width 0) (type default))
-  )
   (wire (pts (xy 200.66 76.2) (xy 205.74 76.2))
     (stroke (width 0) (type default))
@@
   (wire (pts (xy 220.98 63.5) (xy 220.98 60.96))
     (stroke (width 0) (type default))
-  )
-  (rectangle (start 80.01 111.76) (end 132.08 130.81)
-    (stroke (width 0) (type default))
-    (fill (type none))
   )
   (text "https://docs.qmk.fm/#/feature_audio?id=pwm-software"
@@
     (effects (font (size 1.27 1.27)) (justify left bottom))
   )
-  (text "Speaker" (at 80.01 110.49 0)
-    (effects (font (size 1.27 1.27)) (justify left bottom))
-  )
   (label "k20" (at 97.79 62.23 0) (fields_autoplaced)
     (effects (font (size 1.27 1.27)) (justify left bottom))
@@
   (label "k20" (at 124.46 60.96 0) (fields_autoplaced)
     (effects (font (size 1.27 1.27)) (justify left bottom))
-  )
-  (global_label "AUDIO" (shape input) (at 50.8 34.29 180) (fields_autoplaced)
-    (effects (font (size 1.27 1.27)) (justify right))
-    (property "Intersheetrefs" "${INTERSHEET_REFS}" (at 42.2698 34.29 0)
-      (effects (font (size 1.27 1.27)) (justify right) hide)
-    )
-  )
-  (global_label "AUDIO" (shape input) (at 93.98 118.11 180) (fields_autoplaced)
-    (effects (font (size 1.27 1.27)) (justify right))
-    (property "Intersheetrefs" "${INTERSHEET_REFS}" (at 85.4498 118.11 0)
-      (effects (font (size 1.27 1.27)) (justify right) hide)
-    )
   )
   (symbol (lib_id "keyboard_parts:KEYSW") (at 264.16 76.2 0) (mirror y) (unit 1)
@@
         (path "/9538e4ed-27e6-4c37-b989-9859dc0d49e8"
           (reference "K32") (unit 1)
-        )
-      )
-    )
-  )
-  (symbol (lib_id "power:GND") (at 93.98 121.92 0) (mirror y) (unit 1)
-    (in_bom yes) (on_board yes) (dnp no) (fields_autoplaced)
-    (property "Reference" "#PWR01" (at 93.98 128.27 0)
-      (effects (font (size 1.27 1.27)) hide)
-    )
-    (property "Value" "GND" (at 93.98 127 0)
-      (effects (font (size 1.27 1.27)))
-    )
-    (property "Footprint" "" (at 93.98 121.92 0)
-      (effects (font (size 1.27 1.27)) hide)
-    )
-    (property "Datasheet" "" (at 93.98 121.92 0)
-      (effects (font (size 1.27 1.27)) hide)
-    )
-    (pin "1")
-    (instances
-      (project "keyboard_pcb"
-        (path "/9538e4ed-27e6-4c37-b989-9859dc0d49e8"
-          (reference "#PWR01") (unit 1)
-        )
-      )
-      (project "ergodonk_pcb"
-        (path "/ed1aaf15-4e1f-4159-b371-d99b3fb972ad"
-          (reference "#PWR0101") (unit 1)
         )
       )
@@
         )
       )
-    )
-  )
-  (symbol (lib_id "AST1109MLTRQ:AST1109MLTRQ") (at 93.98 118.11 0) (unit 1)
-    (in_bom yes) (on_board yes) (dnp no) (fields_autoplaced)
-    (property "Reference" "LS1" (at 110.49 118.11 0)
-      (effects (font (size 1.524 1.524)) (justify left))
-    )
-    (property "Value" "AST1109MLTRQ_MAL" (at 110.49 121.92 0)
-      (effects (font (size 1.524 1.524)) (justify left))
-    )
-    (property "Footprint" "Cantor_MasterKey:AST1109MLTRQ" (at 101.6 114.554 0)
-      (effects (font (size 1.524 1.524)) hide)
-    )
-    (property "Datasheet" "" (at 93.98 118.11 0)
-      (effects (font (size 1.524 1.524)))
-    )
-    (pin "1")
-    (pin "2")
-    (instances
-      (project "keyboard_pcb"
-        (path "/9538e4ed-27e6-4c37-b989-9859dc0d49e8"
-          (reference "LS1") (unit 1)
-        )
-      )
-      (project "ergodonk_pcb"
-        (path "/ed1aaf15-4e1f-4159-b371-d99b3fb972ad"
-          (reference "LS1") (unit 1)
-        )
-      )

Commit message: Consolidated cantor mx only footprints Removed masterkey footprint library Removed text from tenting puck footprint
Parts:
- J1: footprint Cantor_MasterKey:MJ-4PP-9_Cantor_MX_TX-RX_Crossover -> Cantor_MX:MJ-4PP-9_Cantor_MX_TX-RX_Crossover
- K00, K01, K02, K03, K04, K05, K10, K11, K12, K13, K14, K15, K20, K21, K22, K23, K24, K25, K30, K31, K32: footprint Cantor_MasterKey:CherryMX_ChocV2_1u_DS -> Cantor_MX:CherryMX_ChocV2_1u_DS
- U1: footprint Cantor_MasterKey:Cantor_DS_YAAJ_WeAct_BlackPill_2 -> Cantor_MX:Cantor_DS_YAAJ_WeAct_BlackPill_2
Changed lines of the file:
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@@
       (effects (font (size 1.524 1.524)) hide)
     )
-    (property "Footprint" "Cantor_MasterKey:CherryMX_ChocV2_1u_DS" (at 264.16 76.2 0)
+    (property "Footprint" "Cantor_MX:CherryMX_ChocV2_1u_DS" (at 264.16 76.2 0)
       (effects (font (size 1.524 1.524)) hide)
     )
@@
       (effects (font (size 1.524 1.524)) hide)
     )
-    (property "Footprint" "Cantor_MasterKey:CherryMX_ChocV2_1u_DS" (at 238.76 60.96 0)
+    (property "Footprint" "Cantor_MX:CherryMX_ChocV2_1u_DS" (at 238.76 60.96 0)
       (effects (font (size 1.524 1.524)) hide)
     )
@@
       (effects (font (size 1.524 1.524)) hide)
     )
-    (property "Footprint" "Cantor_MasterKey:CherryMX_ChocV2_1u_DS" (at 137.16 30.48 0)
+    (property "Footprint" "Cantor_MX:CherryMX_ChocV2_1u_DS" (at 137.16 30.48 0)
       (effects (font (size 1.524 1.524)) hide)
     )
@@
       (effects (font (size 1.524 1.524)) hide)
     )
-    (property "Footprint" "Cantor_MasterKey:CherryMX_ChocV2_1u_DS" (at 264.16 45.72 0)
+    (property "Footprint" "Cantor_MX:CherryMX_ChocV2_1u_DS" (at 264.16 45.72 0)
       (effects (font (size 1.524 1.524)) hide)
     )
@@
       (effects (font (size 1.524 1.524)) hide)
     )
-    (property "Footprint" "Cantor_MasterKey:CherryMX_ChocV2_1u_DS" (at 213.36 30.48 0)
+    (property "Footprint" "Cantor_MX:CherryMX_ChocV2_1u_DS" (at 213.36 30.48 0)
       (effects (font (size 1.524 1.524)) hide)
     )
@@
       (effects (font (size 1.524 1.524)) hide)
     )
-    (property "Footprint" "Cantor_MasterKey:CherryMX_ChocV2_1u_DS" (at 187.96 30.48 0)
+    (property "Footprint" "Cantor_MX:CherryMX_ChocV2_1u_DS" (at 187.96 30.48 0)
       (effects (font (size 1.524 1.524)) hide)
     )
@@
       (effects (font (size 1.524 1.524)) hide)
     )
-    (property "Footprint" "Cantor_MasterKey:CherryMX_ChocV2_1u_DS" (at 162.56 45.72 0)
+    (property "Footprint" "Cantor_MX:CherryMX_ChocV2_1u_DS" (at 162.56 45.72 0)
       (effects (font (size 1.524 1.524)) hide)
     )
@@
       (effects (font (size 1.524 1.524)) hide)
     )
-    (property "Footprint" "Cantor_MasterKey:CherryMX_ChocV2_1u_DS" (at 187.96 60.96 0)
+    (property "Footprint" "Cantor_MX:CherryMX_ChocV2_1u_DS" (at 187.96 60.96 0)
       (effects (font (size 1.524 1.524)) hide)
     )
@@
       (effects (font (size 1.27 1.27)))
     )
-    (property "Footprint" "Cantor_MasterKey:Cantor_DS_YAAJ_WeAct_BlackPill_2" (at 71.374 87.122 0)
+    (property "Footprint" "Cantor_MX:Cantor_DS_YAAJ_WeAct_BlackPill_2" (at 71.374 87.122 0)
       (effects (font (size 1.27 1.27)) hide)
     )
@@
       (effects (font (size 1.524 1.524)) hide)
     )
-    (property "Footprint" "Cantor_MasterKey:CherryMX_ChocV2_1u_DS" (at 238.76 30.48 0)
+    (property "Footprint" "Cantor_MX:CherryMX_ChocV2_1u_DS" (at 238.76 30.48 0)
       (effects (font (size 1.524 1.524)) hide)
     )
@@
       (effects (font (size 1.524 1.524)) hide)
     )
-    (property "Footprint" "Cantor_MasterKey:CherryMX_ChocV2_1u_DS" (at 213.36 76.2 0)
+    (property "Footprint" "Cantor_MX:CherryMX_ChocV2_1u_DS" (at 213.36 76.2 0)
       (effects (font (size 1.524 1.524)) hide)
     )
@@
       (effects (font (size 1.524 1.524)))
     )
-    (property "Footprint" "Cantor_MasterKey:MJ-4PP-9_Cantor_MX_TX-RX_Crossover" (at 46.99 115.57 0)
+    (property "Footprint" "Cantor_MX:MJ-4PP-9_Cantor_MX_TX-RX_Crossover" (at 46.99 115.57 0)
       (effects (font (size 1.524 1.524)) hide)
     )
@@
       (effects (font (size 1.524 1.524)) hide)
     )
-    (property "Footprint" "Cantor_MasterKey:CherryMX_ChocV2_1u_DS" (at 137.16 60.96 0)
+    (property "Footprint" "Cantor_MX:CherryMX_ChocV2_1u_DS" (at 137.16 60.96 0)
       (effects (font (size 1.524 1.524)) hide)
     )
@@
       (effects (font (size 1.524 1.524)) hide)
     )
-    (property "Footprint" "Cantor_MasterKey:CherryMX_ChocV2_1u_DS" (at 213.36 60.96 0)
+    (property "Footprint" "Cantor_MX:CherryMX_ChocV2_1u_DS" (at 213.36 60.96 0)
       (effects (font (size 1.524 1.524)) hide)
     )
@@
       (effects (font (size 1.524 1.524)) hide)
     )
-    (property "Footprint" "Cantor_MasterKey:CherryMX_ChocV2_1u_DS" (at 137.16 45.72 0)
+    (property "Footprint" "Cantor_MX:CherryMX_ChocV2_1u_DS" (at 137.16 45.72 0)
       (effects (font (size 1.524 1.524)) hide)
     )
@@
       (effects (font (size 1.524 1.524)) hide)
     )
-    (property "Footprint" "Cantor_MasterKey:CherryMX_ChocV2_1u_DS" (at 162.56 30.48 0)
+    (property "Footprint" "Cantor_MX:CherryMX_ChocV2_1u_DS" (at 162.56 30.48 0)
       (effects (font (size 1.524 1.524)) hide)
     )
@@
       (effects (font (size 1.524 1.524)) hide)
     )
-    (property "Footprint" "Cantor_MasterKey:CherryMX_ChocV2_1u_DS" (at 264.16 60.96 0)
+    (property "Footprint" "Cantor_MX:CherryMX_ChocV2_1u_DS" (at 264.16 60.96 0)
       (effects (font (size 1.524 1.524)) hide)
     )
@@
       (effects (font (size 1.524 1.524)) hide)
     )
-    (property "Footprint" "Cantor_MasterKey:CherryMX_ChocV2_1u_DS" (at 238.76 76.2 0)
+    (property "Footprint" "Cantor_MX:CherryMX_ChocV2_1u_DS" (at 238.76 76.2 0)
       (effects (font (size 1.524 1.524)) hide)
     )
@@
       (effects (font (size 1.524 1.524)) hide)
     )
-    (property "Footprint" "Cantor_MasterKey:CherryMX_ChocV2_1u_DS" (at 238.76 45.72 0)
+    (property "Footprint" "Cantor_MX:CherryMX_ChocV2_1u_DS" (at 238.76 45.72 0)
       (effects (font (size 1.524 1.524)) hide)
     )
@@
       (effects (font (size 1.524 1.524)) hide)
     )
-    (property "Footprint" "Cantor_MasterKey:CherryMX_ChocV2_1u_DS" (at 213.36 45.72 0)
+    (property "Footprint" "Cantor_MX:CherryMX_ChocV2_1u_DS" (at 213.36 45.72 0)
       (effects (font (size 1.524 1.524)) hide)
     )
@@
       (effects (font (size 1.524 1.524)) hide)
     )
-    (property "Footprint" "Cantor_MasterKey:CherryMX_ChocV2_1u_DS" (at 162.56 60.96 0)
+    (property "Footprint" "Cantor_MX:CherryMX_ChocV2_1u_DS" (at 162.56 60.96 0)
       (effects (font (size 1.524 1.524)) hide)
     )
@@
       (effects (font (size 1.524 1.524)) hide)
     )
-    (property "Footprint" "Cantor_MasterKey:CherryMX_ChocV2_1u_DS" (at 187.96 45.72 0)
+    (property "Footprint" "Cantor_MX:CherryMX_ChocV2_1u_DS" (at 187.96 45.72 0)
       (effects (font (size 1.524 1.524)) hide)
     )
@@
       (effects (font (size 1.524 1.524)) hide)
     )
-    (property "Footprint" "Cantor_MasterKey:CherryMX_ChocV2_1u_DS" (at 264.16 30.48 0)
-      (effects (font (size 1.524 1.524)) hide)
-    )
+    (property "Footprint" "Cantor_MX:CherryMX_ChocV2_1u_DS" (at 264.16 30.48 0)
+      (effects (font (size 1.524 1.524)) hide)
+    )
